Commit message: create packages for real model

File: mr2_description/urdf/base/base.gazebo.xacro (robot description, xacro)
@@ -3,5 +3,5 @@
   <xacro:macro name="base_gazebo">
     <gazebo reference="base_link">
-      <selfCollide>true</selfCollide>
+      <selfCollide>false</selfCollide>
       <mu1 value="0.05"/>
       <mu2 value="0.05"/>

File: mr2_description/urdf/legs/leg1.urdf.xacro (robot description, xacro)
@@ -23,5 +23,5 @@
       <inertial>
         <mass value="0.11"/>
-        <inertia ixx="0" ixy="0" ixz="0" iyy="0" iyz="0" izz="0"/>
+        <inertia ixx="0.002" ixy="0" ixz="0" iyy="0.0004" iyz="0" izz="0.003"/>
       </inertial>
     </link>

File: mr2_description/urdf/legs/leg2.urdf.xacro (robot description, xacro)
@@ -26,5 +26,5 @@
         <origin rpy="${M_PI} 0 0" xyz="0 0 0"/>
         <mass value="0.08"/>
-        <inertia ixx="0" ixy="0" ixz="0" iyy="0" iyz="0" izz="0"/>
+        <inertia ixx="0.004" ixy="0" ixz="0" iyy="0.002" iyz="0" izz="0.003"/>
       </inertial>
     </link>

File: mr2_description/urdf/legs/leg3.urdf.xacro (robot description, xacro)
@@ -25,6 +25,6 @@
       <inertial>
         <origin rpy="${M_PI} 0 0" xyz="0 0 0"/>
-        <mass value="0.08"/>
-        <inertia ixx="0" ixy="0" ixz="0" iyy="0" iyz="0" izz="0"/>
+        <mass value="0.4"/>
+        <inertia ixx="0.005" ixy="0" ixz="0" iyy="0.007" iyz="0" izz="0.007"/>
       </inertial>
     </link>
