Commit message: add launch file for real robot

File: mr2_description/robots/mr2.urdf.xacro (robot description, xacro)
@@ -12,17 +12,17 @@
   <!-- Front right leg -->
   <xacro:leg prefix="fr" parent="base_link">
-    <origin rpy="0 0 0" xyz="0.114 0.13 0"/>
+    <origin rpy="${M_PI} 0 0" xyz="0.114 0.13 0"/>
   </xacro:leg>
   <!-- Front left leg -->
   <xacro:leg prefix="fl" parent="base_link">
-    <origin rpy="0 0 ${M_PI}" xyz="-0.114 0.13 0"/>
+    <origin rpy="${M_PI} 0 ${M_PI}" xyz="-0.114 0.13 0"/>
   </xacro:leg>
   <!-- Rear right leg -->
   <xacro:leg prefix="rr" parent="base_link">
-    <origin rpy="0 0 0" xyz="0.114 -0.13 0"/>
+    <origin rpy="${M_PI} 0 0" xyz="0.114 -0.13 0"/>
   </xacro:leg>
   <!-- Rear left leg -->
   <xacro:leg prefix="rl" parent="base_link">
-    <origin rpy="0 0 ${M_PI}" xyz="-0.114 -0.13 0"/>
+    <origin rpy="${M_PI} 0 ${M_PI}" xyz="-0.114 -0.13 0"/>
   </xacro:leg>
   <!-- =============== Transmission ===============-->

File: mr2_description/urdf/legs/leg.urdf.xacro (robot description, xacro)
@@ -11,5 +11,5 @@
     </xacro:leg1>
     <xacro:leg2 prefix="${prefix}" parent="${prefix}_leg1_link">
-      <origin rpy="${M_PI} 0 0" xyz="0.199 0.0215 -0.0152"/>
+      <origin rpy="0 0 0" xyz="0.199 0.0215 0.0152"/>
     </xacro:leg2>
     <xacro:leg3 prefix="${prefix}" parent="${prefix}_leg2_link">

File: mr2_description/urdf/legs/leg1.urdf.xacro (robot description, xacro)
@@ -12,4 +12,5 @@
     <link name="${prefix}_leg1_link">
       <visual>
+        <origin rpy="${M_PI} 0 0" xyz="0 0 0"/>
         <geometry>
           <mesh filename="package://mr2_description/meshes/leg1.STL"/>
@@ -17,4 +18,5 @@
       </visual>
       <collision>
+        <origin rpy="${M_PI} 0 0" xyz="0 0 0"/>
         <geometry>
           <mesh filename="package://mr2_description/meshes/leg1.STL"/>
@@ -22,4 +24,5 @@
       </collision>
       <inertial>
+        <origin rpy="${M_PI} 0 0" xyz="0 0 0"/>
         <mass value="0.11"/>
         <inertia ixx="0.002" ixy="0" ixz="0" iyy="0.0004" iyz="0" izz="0.003"/>

File: mr2_description/urdf/legs/leg2.urdf.xacro (robot description, xacro)
@@ -12,5 +12,5 @@
     <link name="${prefix}_leg2_link">
       <visual>
-        <origin rpy="${M_PI} 0 0" xyz="0 0 0"/>
+        <origin rpy="0 0 0" xyz="0 0 0"/>
         <geometry>
           <mesh filename="package://mr2_description/meshes/leg2.STL"/>
@@ -18,5 +18,5 @@
       </visual>
       <collision>
-        <origin rpy="${M_PI} 0 0" xyz="0 0 0"/>
+        <origin rpy="0 0 0" xyz="0 0 0"/>
         <geometry>
           <mesh filename="package://mr2_description/meshes/leg2.STL"/>
@@ -24,5 +24,5 @@
       </collision>
       <inertial>
-        <origin rpy="${M_PI} 0 0" xyz="0 0 0"/>
+        <origin rpy="0 0 0" xyz="0 0 0"/>
         <mass value="0.08"/>
         <inertia ixx="0.004" ixy="0" ixz="0" iyy="0.002" iyz="0" izz="0.003"/>

File: mr2_description/urdf/legs/leg3.urdf.xacro (robot description, xacro)
@@ -12,5 +12,5 @@
     <link name="${prefix}_leg3_link">
       <visual>
-        <origin rpy="${M_PI} 0 0" xyz="0 0 0"/>
+        <origin rpy="${M_PI} 0 ${M_PI}" xyz="0 0 0"/>
         <geometry>
           <mesh filename="package://mr2_description/meshes/leg3.STL"/>
@@ -18,5 +18,5 @@
       </visual>
       <collision>
-        <origin rpy="${M_PI} 0 0" xyz="0 0 0"/>
+        <origin rpy="${M_PI} 0 ${M_PI}" xyz="0 0 0"/>
         <geometry>
           <mesh filename="package://mr2_description/meshes/leg3.STL"/>
@@ -24,5 +24,5 @@
       </collision>
       <inertial>
-        <origin rpy="${M_PI} 0 0" xyz="0 0 0"/>
+        <origin rpy="${M_PI} 0 ${M_PI}" xyz="0 0 0"/>
         <mass value="0.4"/>
         <inertia ixx="0.005" ixy="0" ixz="0" iyy="0.007" iyz="0" izz="0.007"/>

File: mr2_description/urdf/servo_motors/servo_motors.xacro (robot description, xacro)
@@ -2,4 +2,8 @@
 <robot xmlns:xacro="http://www.ros.org/wiki/xacro">
   <xacro:include filename="$(find mr2_description)/urdf/common.xacro"/>
+  <!-- KRS-3301 ICS -->
+  <xacro:macro name="KRS3301ICS_limit" params="lower_limit:=${-(3*M_PI)/4} upper_limit:=${(3*M_PI)/4}">
+    <limit lower="${lower_limit}" upper="${upper_limit}" effort="${6.0*gravity*0.01}" velocity="${(M_PI/3)/0.14}"/>
+  </xacro:macro>
   <!-- KRS-3302 ICS -->
   <xacro:macro name="KRS3302ICS_limit" params="lower_limit:=${-(3*M_PI)/4} upper_limit:=${(3*M_PI)/4}">
@@ -9,4 +13,8 @@
   <xacro:macro name="KRS3304R2ICS_limit" params="lower_limit:=${-(3*M_PI)/4} upper_limit:=${(3*M_PI)/4}">
     <limit lower="${lower_limit}" upper="${upper_limit}" effort="${13.9*gravity*0.01}" velocity="${(M_PI/3)/0.11}"/>
+  </xacro:macro>
+  <!-- KRS-4034HV ICS -->
+  <xacro:macro name="KRS4034HVICS_limit" params="lower_limit:=${-(3*M_PI)/4} upper_limit:=${(3*M_PI)/4}">
+    <limit lower="${lower_limit}" upper="${upper_limit}" effort="${41.7*gravity*0.01}" velocity="${(M_PI/3)/0.17}"/>
   </xacro:macro>
   <!-- KRS-6003R2HV ICS -->

Commit message: 歩いた

File: mr2_description/robots/mr2.urdf.xacro (robot description, xacro)
@@ -3,4 +3,5 @@
   <xacro:include filename="$(find mr2_description)/urdf/base/base.urdf.xacro"/>
   <xacro:include filename="$(find mr2_description)/urdf/legs/leg.urdf.xacro"/>
+  <xacro:include filename="$(find mr2_description)/urdf/sensors/imu/imu.urdf.xacro"/>
   <!-- =============== Links & Joints =============== -->
   <!-- Base -->
@@ -26,4 +27,9 @@
     <origin rpy="${M_PI} 0 ${M_PI}" xyz="-0.114 -0.13 0"/>
   </xacro:leg>
+  <!-- Sensors -->
+  <!-- IMU -->
+  <xacro:imu id_num="1" parent="base_link">
+    <origin xyz="0 0 0" rpy="0 0 0"/>
+  </xacro:imu>
   <!-- =============== Transmission ===============-->
   <xacro:legs_trans prefix="fr"/>
@@ -44,3 +50,5 @@
   <xacro:legs_gazebo prefix="rr"/>
   <xacro:legs_gazebo prefix="rl"/>
+  <!-- IMU -->
+  <xacro:imu_gazebo id_num="1"/>
 </robot>
