Commit message: add new spider robot

File: mr2_description/urdf/common.xacro (robot description, xacro)
@@ -3,3 +3,9 @@
   <xacro:property name="M_PI" value="3.14159274"/>
   <xacro:property name="gravity" value="9.80665"/>
+  <xacro:macro name="box_inertial" params="mass height width depth">
+    <mass value="${mass}"/>
+    <inertia ixx="${(mass*(width*width + depth*depth))/12}" ixy="0" ixz="0"
+             iyy="${(mass*(height*height + depth*depth))/12}" iyz="0"
+             izz="${(mass*(height*height + width*width))/12}"/>
+  </xacro:macro>
 </robot>

File: mr2_description/urdf/legs/leg1_2.urdf.xacro (robot description, xacro)
@@ -6,5 +6,5 @@
       <xacro:insert_block name="joint_origin"/>
       <axis xyz="0 0 1"/>
-      <xacro:servo_limit/>
+      <xacro:KRS4034HVICS_limit/>
       <parent link="${parent}"/>
       <child link="${prefix}_leg1_link"/>
@@ -12,19 +12,22 @@
     <link name="${prefix}_leg1_link">
       <visual>
-        <origin rpy="${M_PI} 0 0" xyz="0 0 0"/>
+        <origin rpy="0.00000 0.00000 0.00000" xyz="0.00000 0.00000 0.00000"/>
         <geometry>
-          <mesh filename="package://mr2_description/meshes/leg1.STL"/>
+          <mesh filename="package://mr2_description/meshes/leg1_2.STL"/>
         </geometry>
       </visual>
       <collision>
-        <origin rpy="${M_PI} 0 0" xyz="0 0 0"/>
+        <origin rpy="0.00000 0.00000 0.00000" xyz="0.00000 0.00000 0.00000"/>
         <geometry>
-          <mesh filename="package://mr2_description/meshes/leg1.STL"/>
+          <mesh filename="package://mr2_description/meshes/leg1_2.STL"/>
         </geometry>
       </collision>
       <inertial>
-        <origin rpy="${M_PI} 0 0" xyz="0 0 0"/>
-        <mass value="0.11"/>
-        <inertia ixx="0.002" ixy="0" ixz="0" iyy="0.0004" iyz="0" izz="0.003"/>
+        <origin rpy="-0.14190 2.35619 1.42899" xyz="-0.00006 -0.02500 -0.01987"/>
+        <mass value="0.01599"/>
+        <inertia
+          ixx="0.00000569169" ixy="0.00000000000" ixz="0.00000000000"
+          iyy="0.00000586951" iyz="0.00000000000"
+          izz="0.00000587725"/>
       </inertial>
     </link>

File: mr2_description/urdf/legs/leg2_2.urdf.xacro (robot description, xacro)
@@ -5,6 +5,6 @@
     <joint name="${prefix}_leg2_joint" type="revolute">
       <xacro:insert_block name="joint_origin"/>
-      <axis xyz="0 1 0"/>
-      <xacro:servo_limit/>
+      <axis xyz="1 0 0"/>
+      <xacro:KRS4034HVICS_limit/>
       <parent link="${parent}"/>
       <child link="${prefix}_leg2_link"/>
@@ -12,19 +12,22 @@
     <link name="${prefix}_leg2_link">
       <visual>
-        <origin rpy="0 0 0" xyz="0 0 0"/>
+        <origin rpy="0.00000 0.00000 0.00000" xyz="0.00000 0.00000 0.00000"/>
         <geometry>
-          <mesh filename="package://mr2_description/meshes/leg2.STL"/>
+          <mesh filename="package://mr2_description/meshes/leg2_2.STL"/>
         </geometry>
       </visual>
       <collision>
-        <origin rpy="0 0 0" xyz="0 0 0"/>
+        <origin rpy="0.00000 0.00000 0.00000" xyz="0.00000 0.00000 0.00000"/>
         <geometry>
-          <mesh filename="package://mr2_description/meshes/leg2.STL"/>
+          <mesh filename="package://mr2_description/meshes/leg2_2.STL"/>
         </geometry>
       </collision>
       <inertial>
-        <origin rpy="0 0 0" xyz="0 0 0"/>
-        <mass value="0.08"/>
-        <inertia ixx="0.004" ixy="0" ixz="0" iyy="0.002" iyz="0" izz="0.003"/>
+        <origin rpy="0.00000 0.00000 1.57079" xyz="-0.01969 -0.12100 0"/>
+        <mass value="0.23699"/>
+        <inertia
+          ixx="0.00006523998" ixy="0.00000000000" ixz="0.00000000000"
+          iyy="0.00205800016" iyz="0.00000000000"
+          izz="0.00208625265"/>
       </inertial>
     </link>

File: mr2_description/urdf/legs/leg3_2.urdf.xacro (robot description, xacro)
@@ -5,6 +5,6 @@
     <joint name="${prefix}_leg3_joint" type="revolute">
       <xacro:insert_block name="joint_origin"/>
-      <axis xyz="0 1 0"/>
-      <xacro:servo_limit/>
+      <axis xyz="1 0 0"/>
+      <xacro:KRS4034HVICS_limit/>
       <parent link="${parent}"/>
       <child link="${prefix}_leg3_link"/>
@@ -12,19 +12,22 @@
     <link name="${prefix}_leg3_link">
       <visual>
-        <origin rpy="${M_PI} 0 ${M_PI}" xyz="0 0 0"/>
+        <origin rpy="0.00000 0.00000 0.00000" xyz="0.00000 0.00000 0.00000"/>
         <geometry>
-          <mesh filename="package://mr2_description/meshes/leg3.STL"/>
+          <mesh filename="package://mr2_description/meshes/leg3_2.STL"/>
         </geometry>
       </visual>
       <collision>
-        <origin rpy="${M_PI} 0 ${M_PI}" xyz="0 0 0"/>
+        <origin rpy="0.00000 0.00000 0.00000" xyz="0.00000 0.00000 0.00000"/>
         <geometry>
-          <mesh filename="package://mr2_description/meshes/leg3.STL"/>
+          <mesh filename="package://mr2_description/meshes/leg3_2.STL"/>
         </geometry>
       </collision>
       <inertial>
-        <origin rpy="${M_PI} 0 ${M_PI}" xyz="0 0 0"/>
-        <mass value="0.4"/>
-        <inertia ixx="0.005" ixy="0" ixz="0" iyy="0.007" iyz="0" izz="0.007"/>
+        <origin rpy="0.00000 1.59079 -1.57079" xyz="0.01987 0.00114 0.14678"/>
+        <mass value="0.13257"/>
+        <inertia
+          ixx="0.00004387620" ixy="0.00000000000" ixz="0.00000000000"
+          iyy="0.00059834039" iyz="0.00000000000"
+          izz="0.00062747138"/>
       </inertial>
     </link>

File: mr2_description/urdf/sensors/imu/imu.urdf.xacro (robot description, xacro)
@@ -1,9 +1,9 @@
 <?xml version="1.0"?>
 <robot xmlns:xacro="http://www.ros.org/wiki/xacro">
-  <xacro:include filename="$(find omnibot3_description)/urdf/common.xacro"/>
-  <xacro:include filename="$(find omnibot3_description)/urdf/sensors/imu/imu.gazebo.xacro"/>
+  <xacro:include filename="$(find mr2_description)/urdf/common.xacro"/>
+  <xacro:include filename="$(find mr2_description)/urdf/sensors/imu/imu.gazebo.xacro"/>
   <xacro:macro name="imu" params="id_num parent *joint_origin">
     <joint name="imu${id_num}_joint" type="fixed">
-      <insert_block name="joint_origin"/>
+      <xacro:insert_block name="joint_origin"/>
       <parent link="${parent}"/>
       <child link="imu${id_num}_link"/>

File: mr2_description/urdf/servo_motors/servo_motors.xacro (robot description, xacro)
@@ -24,5 +24,5 @@
   <!-- imaginary servo for test -->
   <xacro:macro name="servo_limit" params="lower_limit:=${-(3*M_PI)/4} upper_limit:=${(3*M_PI)/4}">
-    <limit lower="${lower_limit}" upper="${upper_limit}" effort="100" velocity="${(M_PI/3)/0.22}"/>
+    <limit lower="${lower_limit}" upper="${upper_limit}" effort="1000" velocity="${(M_PI/3)/0.22}"/>
   </xacro:macro>
 </robot>
